File: Nucleo_L152RE/ProtoBoard/AA/ProtoBoard.kicad_pcb (KiCad board)
At the start: 2 copper layers, 68.6 x 80.5 mm, 115 parts, among them CON1 USB-MICRO-B, J1 EXT1, J2 EXT2, J3 EXTPower, P1 Power, P10 OW2_A, P11 GND1, P12 I2C1_B, P13 I2C2_B, P14 SW_1_6, P15 WS1, P16 WS2, P17 MS2, P18 WS3, P19 WS4, P2 VinPower, P20 GND2, P21 Hole, P22 MS3, P23 OW3_A, P24 OW4_A, P25 MS4, P26 Hole, P27 Hole, P28 RGB1, P29 Ant, P3 USART2, P30 Hole, P4 SWD Header, P5 USART1, P6 MS1, P7 I2C1_A, P8 I2C2_A, P9 OW1_A, Q1 SI2323DS, SW1 MomentarySwitch, U2 Nucleo-L152RE-CN7, U3 Nucleo-L152RE-CN10, U5 MT3329_GPS, U6 S25FL127S, U7 RFM69HW

Commit message: Fixed Flash and Pmos footprints.  Added symbol part for schematic.
Parts:
- removed REF**: Symbol_OSHW-Logo_SilkScreen, Symbols:Symbol_OSHW-Logo_SilkScreen
- added S1: OSHW Symbol, Symbols:Symbol_OSHW-Logo_SilkScreen, F.Cu at (137.0, 72.4)
- Q1: footprint SMD_Packages:SOT-323 -> nucleo:TO-236
- U6: footprint SMD_Packages:SOIC-8-N -> nucleo:SOIC-8-FLASH
- moved Q1 1.01 mm to (135.8, 111.3)
- moved C1 0.98 mm to (135.5, 113.5)
- moved JP21 0.31 mm to (153.8, 51.2)
- moved JP20 0.28 mm to (152.5, 51.2)
- moved C8 0.15 mm to (150.9, 57.0)
Routing:
- net GND: track 528.7 -> 536.2 mm, vias 30 -> 32
- net /VIN_Trig: track 23.2 -> 29.3 mm
- net +15V: track 11.0 -> 16.5 mm
- net Net-(Q1-Pad3): track 3.45 -> 8.49 mm
- net Net-(C1-Pad1): track 4.01 -> 4.86 mm
Other:
- board text added: "3.3v only"
- board text added: "B"
- board text added: "CC SA"
- board text added: "Dustin Reynolds STM32 Sensor Shield Nucleo-L152RE"
- board text added: "E5V 5.0v only NEG"
- board text added: "E5V 5.0v only POS"
- board text added: "Ext Bus Pin Out 1. 3.3v 2. Gnd 3. SPI CS 4. SPI CLK 5. SPI MOSI 6. SPI MISO 7. ADC 8. GPIO/DAC (3.3V only)"
- board text added: "Ext Power Connection 1. MotionSense3 2. MotionSense4 3. StatusLed4 4. SPI CLK 5. SPI MOSI 6. SPI MISO 7. E5V 8. Gnd"
- board text added: "G"
- board text added: "I2C Bus 1"
- board text added: "MS2 3.3v only"
- board text added: "OneWire1"
- board text added: "OneWire2"
- board text added: "R"
- board text added: "RF ID: ___________________ SN: ___________________"
- board text added: "Sig"
- board text added: "YMD: 20150405"
- board text removed: "Dustin Reynolds"
- board text removed: "E5V 5.0v only Pos Neg"
- board text removed: "RF ID: __________"
- board text removed: "Revision ___________"
- board text removed: "STM32 Sensor Shield"
- board text removed: "Serial Number: __________"
