File: Nucleo_L152RE/ProtoBoard/AA/ProtoBoard.sch (KiCad schematic (older format))
At the start: 116 parts, among them CON1 USB-MICRO-B, J1 EXT1, J2 EXT2, J3 EXTPower, P1 Power, P10 OW2_A, P11 GND1, P12 I2C1_B, P13 I2C2_B, P14 SW_1_6, P15 WS1, P16 WS2, P17 MS2, P18 WS3, P19 WS4, P2 VinPower, P20 GND2, P21 Hole, P22 MS3, P23 OW3_A, P24 OW4_A, P25 MS4, P26 Hole, P27 Hole, P28 RGB1, P29 Ant, P3 USART2, P30 Hole, P4 SWD Header, P5 USART1, P6 MS1, P7 I2C1_A, P8 I2C2_A, P9 OW1_A, Q1 SI2323DS, SW1 MomentarySwitch, U2 Nucleo-L152RE-CN7, U3 Nucleo-L152RE-CN10, U5 MT3329_GPS, U6 S25FL127S, U7 RFM69HW

Commit message: Found 5 unconnected pins on Nucleo L152RE, so I've added an Errata and deleted the wires for the effected nets.
Connections:
- wire segments 322 -> 317
Other:
- note added: "Rev AA Errata 4-26-2015:\nU2: Pin 9, 11 No Connection\nU3: Pin 10: No Connection\n Pin 36: VDD (same as U2 Pin 5\n Pin 38: GND"
- moved on the sheet: CON1, JP6, JP7, JP8, JP9, R11, R12, R5

Commit message: Adding notes to schematic and board layout to indicate the very broken wireless module interface.  New board will need to be created to fix the issue.
Other:
- note added: "Chip has the wrong pinout!\nNumbering Should have \nbeen correct (9 across from 8)"
- note added: "Rev AA Errata 4-26-2015:\nU2: Pin 9, 11 No Connection\nU3: Pin 10: No Connection\n Pin 36: No Connection\n Pin 38: No Connection"
- note removed: "Rev AA Errata 4-26-2015:\nU2: Pin 9, 11 No Connection\nU3: Pin 10: No Connection\n Pin 36: VDD (same as U2 Pin 5\n Pin 38: GND"
- moved on the sheet: U7
Changed lines of the file:
@@
 L RFM69HW U7
 U 1 1 55169D6F
-P 14550 1600
-F 0 "U7" H 14550 2050 60  0000 C CNN
-F 1 "RFM69HW" H 14450 1150 60  0000 C CNN
-F 2 "nucleo:RFM69HW" H 14550 1600 60  0001 C CNN
-F 3 "" H 14550 1600 60  0000 C CNN
-F 4 "RFM69HW 915MHz" H 14550 1600 60  0001 C CNN "Ebay"
-	1    14550 1600
+P 14750 800
+F 0 "U7" H 14750 1250 60  0000 C CNN
+F 1 "RFM69HW" H 14650 350 60  0000 C CNN
+F 2 "nucleo:RFM69HW" H 14750 800 60  0001 C CNN
+F 3 "" H 14750 800 60  0000 C CNN
+F 4 "RFM69HW 915MHz" H 14750 800 60  0001 C CNN "Ebay"
+	1    14750 800
 	1    0    0    -1
 $EndComp
@@
 	7700 4450 7700 6150
 Text Notes 550  950  0    59   ~ 0
-Rev AA Errata 4-26-2015:\nU2: Pin 9, 11 No Connection\nU3: Pin 10: No Connection\n       Pin 36: VDD (same as U2 Pin 5\n       Pin 38: GND
+Rev AA Errata 4-26-2015:\nU2: Pin 9, 11 No Connection\nU3: Pin 10: No Connection\n       Pin 36: No Connection\n       Pin 38: No Connection
+Text Notes 14000 2450 0    59   ~ 0
+Chip has the wrong pinout!\nNumbering Should have \nbeen correct (9 across from 8)
 $EndSCHEMATC

Commit message: Making more changes on Rev AB. Found that the voltage measurement circuit didn't work as expected, so it has been replaced with a voltage divider.  Removing second Ethernet port since they take up a lot of space and the utilization of it would probably be pretty low.  Corrected many errors from Rev AA.
Other:
- note added: "Voltage at VIN_Trig too high"
- moved on the sheet: U7
Changed lines of the file:
@@
 L RFM69HW U7
 U 1 1 55169D6F
-P 14750 800
-F 0 "U7" H 14750 1250 60  0000 C CNN
-F 1 "RFM69HW" H 14650 350 60  0000 C CNN
-F 2 "nucleo:RFM69HW" H 14750 800 60  0001 C CNN
-F 3 "" H 14750 800 60  0000 C CNN
-F 4 "RFM69HW 915MHz" H 14750 800 60  0001 C CNN "Ebay"
-	1    14750 800
+P 14550 1600
+F 0 "U7" H 14550 2050 60  0000 C CNN
+F 1 "RFM69HW" H 14450 1150 60  0000 C CNN
+F 2 "nucleo:RFM69HW" H 14550 1600 60  0001 C CNN
+F 3 "" H 14550 1600 60  0000 C CNN
+F 4 "RFM69HW 915MHz" H 14550 1600 60  0001 C CNN "Ebay"
+	1    14550 1600
 	1    0    0    -1
 $EndComp
@@
 Text Notes 14000 2450 0    59   ~ 0
 Chip has the wrong pinout!\nNumbering Should have \nbeen correct (9 across from 8)
+Text Notes 600  7200 0    59   ~ 0
+Voltage at VIN_Trig too high
 $EndSCHEMATC
