File: Nucleo_L152RE/ProtoBoard/AB/Sensors.sch (KiCad schematic (older format))
At the start: 83 parts, among them P32 SWBUS1, P36 USART2, P37 SWD Header, P38 RGB1, P39 USART1, P40 MS1, P41 MS3, P42 MS2, P43 MS4, P44 RLY1, P45 OW1_A, P46 I2C1_A, P47 I2C2_A, P48 RLY2, P49 I2C1_B, P50 I2C2_B, P51 FET_SW1, P52 WS1, P53 OW2_A, P54 OW3_A, P56 WS2, P57 WS2, Q1 BSS123-7-F, Q2 BSS123-7-F, SW1 MomentarySwitch, SW2 ResetSwitch

Commit message: Finished AB board.
Connections:
- net at D4.2 (A): now also R17.2; no longer R15.2
- net at D5.2 (A): now also R18.2; no longer R16.2
- net at D2.2 (A): now also R15.2; no longer R17.2
- net at D3.2 (A): now also R16.2; no longer R18.2
Other:
- note added: "30V 1A max"
- note added: "Nucleo_LED connected to Red"
- note removed: "Future boards can be powered\nusing this pin"
- moved on the sheet: R15, R16, R17, R18
Changed lines of the file:
@@
 Sheet 4 5
 Title "Expansion Board For STM32 Nucleo-L152RE"
-Date "Sunday, May 31, 2015"
-Rev "AB - Final Draft"
+Date "Monday, June 01, 2015"
+Rev "AB"
 Comp "Open Source Hardware"
 Comment1 "MIT License"
@@
 L R_Small R15
 U 1 1 555AC215
-P 1300 3150
-F 0 "R15" H 1330 3170 50  0000 L CNN
-F 1 "1K" H 1330 3110 50  0000 L CNN
-F 2 "Resistors_SMD:R_0603_HandSoldering" H 1300 3150 60  0001 C CNN
-F 3 "" H 1300 3150 60  0000 C CNN
-F 4 "P1.0KGCT-ND" H 1300 3150 60  0001 C CNN "Digikey Part Number"
-F 5 "ERJ-3GEYJ102V" H 2900 2200 60  0001 C CNN "MFG"
-	1    1300 3150
+P 1300 3650
+F 0 "R15" H 1330 3670 50  0000 L CNN
+F 1 "1K" H 1330 3610 50  0000 L CNN
+F 2 "Resistors_SMD:R_0603_HandSoldering" H 1300 3650 60  0001 C CNN
+F 3 "" H 1300 3650 60  0000 C CNN
+F 4 "P1.0KGCT-ND" H 1300 3650 60  0001 C CNN "Digikey Part Number"
+F 5 "ERJ-3GEYJ102V" H 2900 2700 60  0001 C CNN "MFG"
+	1    1300 3650
 	0    -1   -1   0
 $EndComp
@@
 L R_Small R16
 U 1 1 555AC21E
-P 1300 3400
-F 0 "R16" H 1330 3420 50  0000 L CNN
-F 1 "1k" H 1330 3360 50  0000 L CNN
-F 2 "Resistors_SMD:R_0603_HandSoldering" H 1300 3400 60  0001 C CNN
-F 3 "" H 1300 3400 60  0000 C CNN
-F 4 "P1.0KGCT-ND" H 1300 3400 60  0001 C CNN "Digikey Part Number"
-F 5 "ERJ-3GEYJ102V" H 2900 2200 60  0001 C CNN "MFG"
-	1    1300 3400
+P 1300 3900
+F 0 "R16" H 1330 3920 50  0000 L CNN
+F 1 "1k" H 1330 3860 50  0000 L CNN
+F 2 "Resistors_SMD:R_0603_HandSoldering" H 1300 3900 60  0001 C CNN
+F 3 "" H 1300 3900 60  0000 C CNN
+F 4 "P1.0KGCT-ND" H 1300 3900 60  0001 C CNN "Digikey Part Number"
+F 5 "ERJ-3GEYJ102V" H 2900 2700 60  0001 C CNN "MFG"
+	1    1300 3900
 	0    -1   -1   0
 $EndComp
@@
 Text Notes 8950 4250 0    39   ~ 0
 PWM
-Text Notes 650  3000 0    39   ~ 0
-Future boards can be powered\nusing this pin
 $Comp
 L R_Small R17
 U 1 1 555AC2A1
-P 1300 3650
-F 0 "R17" H 1330 3670 50  0000 L CNN
-F 1 "1k" H 1330 3610 50  0000 L CNN
-F 2 "Resistors_SMD:R_0603_HandSoldering" H 1300 3650 60  0001 C CNN
-F 3 "" H 1300 3650 60  0000 C CNN
-F 4 "P1.0KGCT-ND" H 1300 3650 60  0001 C CNN "Digikey Part Number"
-	1    1300 3650
+P 1300 3150
+F 0 "R17" H 1330 3170 50  0000 L CNN
+F 1 "1k" H 1330 3110 50  0000 L CNN
+F 2 "Resistors_SMD:R_0603_HandSoldering" H 1300 3150 60  0001 C CNN
+F 3 "" H 1300 3150 60  0000 C CNN
+F 4 "P1.0KGCT-ND" H 1300 3150 60  0001 C CNN "Digikey Part Number"
+	1    1300 3150
 	0    -1   -1   0
 $EndComp
@@
 L R_Small R18
 U 1 1 555AC2B6
-P 1300 3900
-F 0 "R18" H 1330 3920 50  0000 L CNN
-F 1 "1k" H 1330 3860 50  0000 L CNN
-F 2 "Resistors_SMD:R_0603_HandSoldering" H 1300 3900 60  0001 C CNN
-F 3 "" H 1300 3900 60  0000 C CNN
-F 4 "P1.0KGCT-ND" H 1300 3900 60  0001 C CNN "Digikey Part Number"
-F 5 "ERJ-3GEYJ102V" H 2900 2200 60  0001 C CNN "MFG"
-	1    1300 3900
+P 1300 3400
+F 0 "R18" H 1330 3420 50  0000 L CNN
+F 1 "1k" H 1330 3360 50  0000 L CNN
+F 2 "Resistors_SMD:R_0603_HandSoldering" H 1300 3400 60  0001 C CNN
+F 3 "" H 1300 3400 60  0000 C CNN
+F 4 "P1.0KGCT-ND" H 1300 3400 60  0001 C CNN "Digikey Part Number"
+F 5 "ERJ-3GEYJ102V" H 2900 1700 60  0001 C CNN "MFG"
+	1    1300 3400
 	0    -1   -1   0
 $EndComp
@@
 	1    0    0    -1
 $EndComp
-Text Notes 1950 3700 0    39   ~ 0
+Text Notes 1950 3250 0    39   ~ 0
 StatusLed3 Shares pin with \nGPS Enable
-Text Notes 1950 3900 0    39   ~ 0
+Text Notes 1950 3450 0    39   ~ 0
 StatusLed4 Shares pin with \nEXT 3.3V en
 Text Notes 3250 750  0    59   ~ 0
@@
 	1450 1000 2300 1000
 Wire Wire Line
-	1700 3150 1850 3150
-Wire Wire Line
-	1400 3150 1500 3150
-Wire Wire Line
-	1500 3400 1400 3400
+	1400 3650 1500 3650
+Wire Wire Line
+	1500 3900 1400 3900
 Wire Wire Line
 	2150 2350 2300 2350
@@
 Connection ~ 6850 5100
 Wire Wire Line
-	1400 3650 1500 3650
-Wire Wire Line
-	1700 3150 1700 3900
-Connection ~ 1700 3400
+	1400 3150 1500 3150
+Connection ~ 1700 3900
 Wire Wire Line
 	1850 3150 1850 3200
 Wire Wire Line
-	1400 3900 1500 3900
-Connection ~ 1700 3650
+	1400 3400 1500 3400
+Connection ~ 1700 3150
 Wire Wire Line
 	9750 3750 9750 4000
@@
 F1 "Modules.sch" 59
 $EndSheet
+Text GLabel 1200 3650 0    59   Input ~ 0
+StatusLed1
+Text GLabel 1200 3900 0    59   Input ~ 0
+StatusLed2
 Text GLabel 1200 3150 0    59   Input ~ 0
-StatusLed1
+StatusLed3
 Text GLabel 1200 3400 0    59   Input ~ 0
-StatusLed2
-Text GLabel 1200 3650 0    59   Input ~ 0
-StatusLed3
-Text GLabel 1200 3900 0    59   Input ~ 0
 StatusLed4
 Text GLabel 1300 2350 0    59   Input ~ 0
@@
 Wire Wire Line
 	4800 4100 4700 4100
+Wire Wire Line
+	1700 3150 1700 3900
+Wire Wire Line
+	1700 3150 1850 3150
+Connection ~ 1700 3400
+Connection ~ 1700 3650
+Text Notes 700  1700 0    59   ~ 0
+Nucleo_LED connected to Red
+Text Notes 3200 2450 0    59   ~ 0
+30V 1A max
 $EndSCHEMATC

Commit message: Updated MFG part numbers on schematic for BOM generation.
Parts:
- Q1, Q2: MFG (none) -> BSS123-7-F
- RLY1: MFG (none) -> TQ2SA-3V
Changed lines of the file:
@@
 F 2 "nucleo:SOT23-3" H 4100 3475 50  0001 L CIN
 F 3 "" H 4100 3625 50  0000 L CNN
+F 4 "BSS123-7-F" H 3900 3550 60  0001 C CNN "MFG"
 	1    3900 3550
 	1    0    0    -1
@@
 F 2 "nucleo:Relay_SMD" H 4850 2920 59  0001 C CNN
 F 3 "" H 4200 2790 59  0000 C CNN
+F 4 "TQ2SA-3V" H 4200 2950 60  0001 C CNN "MFG"
 	1    4200 2950
 	1    0    0    -1
@@
 F 2 "nucleo:SOT23-3" H 4450 4525 50  0001 L CIN
 F 3 "" H 4450 4675 50  0000 L CNN
+F 4 "BSS123-7-F" H 4250 4600 60  0001 C CNN "MFG"
 	1    4250 4600
 	1    0    0    -1
